File: WG-Segment/WG-Segment.kicad_pcb (KiCad board)
At the start: 4 copper layers, 99.8 x 99.8 mm, 140 parts, among them J101 Conn_01x02, J102 Conn_02x04_Odd_Even, J201 Conn_01x03, J202 Conn_01x02, J203 Conn_01x04, J501 Conn_01x02, J502 Conn_01x02, J503 Conn_01x02, J504 Conn_01x02, J505 Conn_01x02, J506 Conn_01x02, J507 Conn_01x02, J508 Conn_01x02, J509 Conn_01x02, J510 Conn_01x02, J511 Conn_01x02, J512 Conn_01x02, J513 Conn_01x02, J514 Conn_01x02, J515 Conn_01x02, J516 Conn_01x02, J517 Conn_01x02, J518 Conn_01x02, J519 Conn_01x02, J520 Conn_01x02, J521 Conn_01x02, J522 Conn_01x02, J523 Conn_01x02, J524 Conn_01x02, J525 Conn_01x02, SW201 SPST-NO, U201 W25Q16JV, U202 RP2040, U301 AP63200WU, U302 MIC5504-3.3YM5, U303 REF3033, U401 SN74LV1T34DCK, U501 SN74LV4051A, U502 SN74LV4051A, U503 SN74LV4051A, U504 SN74LV4051A, Y201 12MHz

Commit message: Add LCSC part numbers
Parts:
- removed C308: 100p, Capacitor_SMD:C_0402_1005Metric_Pad0.74x0.62mm_HandSolder
- removed U303: REF3033, Package_TO_SOT_SMD:SOT-23
- C305, C306: value 1u/10V -> 1u
- C307: value 470n -> 100p
- R301: value 157k -> 120k
- R302: value 30k -> 22k
- moved C307 43.5 mm to (110.4, 67.4), turned to 90 degrees
Connections:
- C212 pad 1: VREF -> +3V3
- C307 pad 2: GND -> Net-(U301-FB)
- J501 pad 1: VREF -> +3V3
- J502 pad 1: VREF -> +3V3
- J503 pad 1: VREF -> +3V3
- J504 pad 1: VREF -> +3V3
- J505 pad 1: VREF -> +3V3
- J506 pad 1: VREF -> +3V3
- J507 pad 1: VREF -> +3V3
- J508 pad 1: VREF -> +3V3
- J509 pad 1: VREF -> +3V3
- J510 pad 1: VREF -> +3V3
- J511 pad 1: VREF -> +3V3
- J512 pad 1: VREF -> +3V3
- J513 pad 1: VREF -> +3V3
- J514 pad 1: VREF -> +3V3
- J515 pad 1: VREF -> +3V3
- J516 pad 1: VREF -> +3V3
- J517 pad 1: VREF -> +3V3
- J518 pad 1: VREF -> +3V3
- J519 pad 1: VREF -> +3V3
- J520 pad 1: VREF -> +3V3
- J521 pad 1: VREF -> +3V3
- J522 pad 1: VREF -> +3V3
- J523 pad 1: VREF -> +3V3
- J524 pad 1: VREF -> +3V3
- J525 pad 1: VREF -> +3V3
- U202 pad 43: VREF -> +3V3
Routing:
- net VREF: track 738.0 -> 0.00 mm
- net +3V3: track 112.4 -> 845.6 mm, vias 8 -> 9
- net +5V: track 78.6 -> 75.3 mm, vias 247 -> 244
- net GND: track 32.5 -> 30.8 mm, vias 360 -> 359
