File: WG-Segment/cpu.kicad_sch (KiCad schematic)
At the start: 28 parts, among them J201 Conn_01x03, J202 Conn_01x02, J203 Conn_01x04, SW201 SPST-NO, U201 W25Q16JV, U202 RP2040, Y201 12MHz

Commit message: Updates for smoother JLCPCB ordering
Connections:
- net VREF is gone; now on net +3V3: C212.1, U202.43 (ADC_AVDD)
Other:
- note added: "Change this for custom reference voltage"
Changed lines of the file:
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@@
     (effects (font (size 1.27 1.27)) (justify left bottom))
+  )
+  (text "Change this for custom reference voltage" (at 212.09 50.8 0)
+    (effects (font (size 0.635 0.635)) (justify left bottom))
   )
   (text "Possibly could\nbe removed" (at 66.04 85.09 0)
@@
   (label "USB_D+" (at 114.3 68.58 0) (fields_autoplaced)
     (effects (font (size 1.27 1.27)) (justify left bottom))
-  )
-  (global_label "VREF" (shape input) (at 209.55 50.8 0) (fields_autoplaced)
-    (effects (font (size 1.27 1.27)) (justify left))
-    (property "Intersheetrefs" "${INTERSHEET_REFS}" (at 217.1314 50.8 0)
-      (effects (font (size 1.27 1.27)) (justify left) hide)
-    )
   )
   (hierarchical_label "MUX_A" (shape output) (at 191.77 88.9 0) (fields_autoplaced)
@@
         )
       )
+    )
+  )
+  (symbol (lib_id "power:+3V3") (at 209.55 50.8 0) (unit 1)
+    (in_bom yes) (on_board yes) (dnp no) (fields_autoplaced)
+    (property "Reference" "#PWR0201" (at 209.55 54.61 0)
+      (effects (font (size 1.27 1.27)) hide)
+    )
+    (property "Value" "+3V3" (at 209.55 45.72 0)
+      (effects (font (size 1.27 1.27)))
+    )
+    (property "Footprint" "" (at 209.55 50.8 0)
+      (effects (font (size 1.27 1.27)) hide)
+    )
+    (property "Datasheet" "" (at 209.55 50.8 0)
+      (effects (font (size 1.27 1.27)) hide)
+    )
+    (pin "1")
+    (instances
+      (project "WG-Segment"
+        (path "/9a5339e6-f970-4986-a2cb-f70ab323b7e1/1e0e1cdf-3136-4548-bd2e-0b31b8fba863"
+          (reference "#PWR0201") (unit 1)
+        )
+      )

Commit message: Add LCSC part numbers
Parts:
- C201, C202, C205, C206, C207, C208, C209, C210, C211, C212, C213: LCSC Part (none) -> C1525
- C203, C204: LCSC Part (none) -> C52923; Manufacturer (none) -> Samsung Electro-Mechanics; Part Number (none) -> CL05A105KA5NQNC
- C214, C215: LCSC Part (none) -> C1548
- R201: LCSC Part (none) -> C25908
- R204: LCSC Part (none) -> C25744
- R205, R206: LCSC Part (none) -> C11702
- U201: LCSC Part (none) -> C131025
- U202: LCSC Part (none) -> C2040
- Y201: LCSC Part (none) -> C20625731
Changed lines of the file:
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@@
+      (effects (font (size 1.27 1.27)) hide)
+    )
+    (property "LCSC Part" "C1525" (at 266.7 39.37 0)
       (effects (font (size 1.27 1.27)) hide)
     )
@@
     )
     (property "Desc" "CAP CER 15pF 10V 0402" (at 41.91 138.43 0)
+      (effects (font (size 1.27 1.27)) hide)
+    )
+    (property "LCSC Part" "C1548" (at 41.91 138.43 0)
       (effects (font (size 1.27 1.27)) hide)
     )
@@
       (effects (font (size 1.27 1.27)) hide)
     )
+    (property "LCSC Part" "C25744" (at 67.31 83.82 0)
+      (effects (font (size 1.27 1.27)) hide)
+    )
     (pin "1")
     (pin "2")
@@
       (effects (font (size 1.27 1.27)) hide)
     )
+    (property "LCSC Part" "C1548" (at 41.91 153.67 0)
+      (effects (font (size 1.27 1.27)) hide)
+    )
     (pin "1")
     (pin "2")
@@
       (effects (font (size 1.27 1.27)) hide)
     )
+    (property "LCSC Part" "C1525" (at 254 39.37 0)
+      (effects (font (size 1.27 1.27)) hide)
+    )
     (pin "1")
     (pin "2")
@@
     )
     (property "Manufacturer" "Winbond Electronics" (at 41.91 96.52 0)
+      (effects (font (size 1.27 1.27)) hide)
+    )
+    (property "LCSC Part" "C131025" (at 41.91 96.52 0)
       (effects (font (size 1.27 1.27)) hide)
     )
@@
     )
     (property "Part Number" "RP2040" (at 160.02 99.06 0)
+      (effects (font (size 1.27 1.27)) hide)
+    )
+    (property "LCSC Part" "C2040" (at 160.02 99.06 0)
       (effects (font (size 1.27 1.27)) hide)
     )
@@
       (effects (font (size 1.27 1.27)) hide)
     )
+    (property "LCSC Part" "C1525" (at 137.16 39.37 0)
+      (effects (font (size 1.27 1.27)) hide)
+    )
     (pin "1")
     (pin "2")
@@
       (effects (font (size 1.27 1.27)) hide)
     )
-    (property "Part Number" "" (at 179.07 39.37 0)
-      (effects (font (size 1.27 1.27)) hide)
-    )
-    (property "Manufacturer" "" (at 179.07 39.37 0)
+    (property "Part Number" "CL05A105KA5NQNC" (at 179.07 39.37 0)
+      (effects (font (size 1.27 1.27)) hide)
+    )
+    (property "Manufacturer" "Samsung Electro-Mechanics" (at 179.07 39.37 0)
       (effects (font (size 1.27 1.27)) hide)
     )
@@
       (effects (font (size 1.27 1.27)) hide)
     )
+    (property "LCSC Part" "C52923" (at 179.07 39.37 0)
+      (effects (font (size 1.27 1.27)) hide)
+    )
     (pin "1")
     (pin "2")
@@
       (effects (font (size 1.27 1.27)) hide)
     )
-    (property "Part Number" "" (at 148.59 39.37 0)
-      (effects (font (size 1.27 1.27)) hide)
-    )
-    (property "Manufacturer" "" (at 148.59 39.37 0)
+    (property "Part Number" "CL05A105KA5NQNC" (at 148.59 39.37 0)
+      (effects (font (size 1.27 1.27)) hide)
+    )
+    (property "Manufacturer" "Samsung Electro-Mechanics" (at 148.59 39.37 0)
       (effects (font (size 1.27 1.27)) hide)
     )
@@
       (effects (font (size 1.27 1.27)) hide)
     )
+    (property "LCSC Part" "C52923" (at 148.59 39.37 0)
+      (effects (font (size 1.27 1.27)) hide)
+    )
     (pin "1")
     (pin "2")
@@
       (effects (font (size 1.27 1.27)) hide)
     )
+    (property "LCSC Part" "C1525" (at 203.2 39.37 0)
+      (effects (font (size 1.27 1.27)) hide)
+    )
     (pin "1")
     (pin "2")
@@
     )
     (property "Desc" "CAP CER 0.1uF 10V 0402" (at 205.74 54.61 0)
+      (effects (font (size 1.27 1.27)) hide)
+    )
+    (property "LCSC Part" "C1525" (at 205.74 54.61 0)
       (effects (font (size 1.27 1.27)) hide)
     )
@@
       (effects (font (size 1.27 1.27)) hide)
     )
+    (property "LCSC Part" "C11702" (at 74.93 88.9 0)
+      (effects (font (size 1.27 1.27)) hide)
+    )
     (pin "2")
     (pin "1")
@@
       (effects (font (size 1.27 1.27)) hide)
     )
+    (property "LCSC Part" "C1525" (at 228.6 39.37 0)
+      (effects (font (size 1.27 1.27)) hide)
+    )
     (pin "1")
     (pin "2")
@@
       (effects (font (size 1.27 1.27)) hide)
     )
+    (property "LCSC Part" "C1525" (at 241.3 39.37 0)
+      (effects (font (size 1.27 1.27)) hide)
+    )
     (pin "1")
     (pin "2")
@@
     )
     (property "Desc" "CAP CER 0.1uF 10V 0402" (at 24.13 85.09 0)
+      (effects (font (size 1.27 1.27)) hide)
+    )
+    (property "LCSC Part" "C1525" (at 24.13 85.09 0)
       (effects (font (size 1.27 1.27)) hide)
     )
@@
       (effects (font (size 1.27 1.27)) hide)
     )
+    (property "LCSC Part" "C20625731" (at 41.91 146.05 0)
+      (effects (font (size 1.27 1.27)) hide)
+    )
     (pin "2")
     (pin "1")
@@
       (effects (font (size 1.27 1.27)) hide)
     )
+    (property "LCSC Part" "C25908" (at 127 57.15 0)
+      (effects (font (size 1.27 1.27)) hide)
+    )
     (pin "2")
     (pin "1")
@@
     )
     (property "Desc" "CAP CER 0.1uF 10V 0402" (at 190.5 39.37 0)
+      (effects (font (size 1.27 1.27)) hide)
+    )
+    (property "LCSC Part" "C1525" (at 190.5 39.37 0)
       (effects (font (size 1.27 1.27)) hide)
     )
@@
       (effects (font (size 1.27 1.27)) hide)
     )
+    (property "LCSC Part" "C11702" (at 57.15 149.86 0)
+      (effects (font (size 1.27 1.27)) hide)
+    )
     (pin "2")
     (pin "1")
@@
       (effects (font (size 1.27 1.27)) hide)
     )
+    (property "LCSC Part" "C1525" (at 215.9 39.37 0)
+      (effects (font (size 1.27 1.27)) hide)
+    )
     (pin "1")
     (pin "2")
@@
       (effects (font (size 1.27 1.27)) hide)
     )
+    (property "LCSC Part" "C1525" (at 125.73 39.37 0)
+      (effects (font (size 1.27 1.27)) hide)
+    )
