File: WG-Segment/power.kicad_sch (KiCad schematic)
At the start: 15 parts, among them U301 AP63200WU, U302 MIC5504-3.3YM5

Commit message: Add LCSC part numbers
Parts:
- C301: LCSC Part (none) -> C1525
- C302: LCSC Part (none) -> C15850; Manufacturer Murata -> Samsung Electro-Mechanics; Part Number GRM21BR61E106KA73L -> CL21A106KAYNNNE
- C303, C304: LCSC Part (none) -> C45783; Part Number CL21A226MPQNNNE -> CL21A226MAQNNNE
- C305, C306: value 1u/10V -> 1u; LCSC Part (none) -> C52923; Part Number CL05A105KP5NNNC -> CL05A105KA5NQNC
- C307: renamed from C308; LCSC Part (none) -> C1546
- D301: LCSC Part (none) -> C8678
- D302: LCSC Part (none) -> C2286
- R301: LCSC Part (none) -> C25750
- R302: LCSC Part (none) -> C25768
- R303: LCSC Part (none) -> C25117
- U301: LCSC Part (none) -> C2071868
- U302: LCSC Part (none) -> C88419
Changed lines of the file:
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@@
       (effects (font (size 1.27 1.27)) (justify left))
     )
-    (property "Value" "1u/10V" (at 76.2 130.81 0)
+    (property "Value" "1u" (at 76.2 130.81 0)
       (effects (font (size 1.27 1.27)) (justify left))
     )
@@
       (effects (font (size 1.27 1.27)) hide)
     )
-    (property "Part Number" "CL05A105KP5NNNC" (at 72.39 129.54 0)
+    (property "Part Number" "CL05A105KA5NQNC" (at 72.39 129.54 0)
       (effects (font (size 1.27 1.27)) hide)
     )
@@
       (effects (font (size 1.27 1.27)) hide)
     )
+    (property "LCSC Part" "C52923" (at 72.39 129.54 0)
+      (effects (font (size 1.27 1.27)) hide)
+    )
     (pin "1")
     (pin "2")
@@
     )
     (property "Manufacturer" "Microchip Technology" (at 96.52 127 0)
+      (effects (font (size 1.27 1.27)) hide)
+    )
+    (property "LCSC Part" "C88419" (at 96.52 127 0)
       (effects (font (size 1.27 1.27)) hide)
     )
@@
       (effects (font (size 1.27 1.27)) hide)
     )
-    (property "Part Number" "GRM21BR61E106KA73L" (at 96.52 74.93 0)
-      (effects (font (size 1.27 1.27)) hide)
-    )
-    (property "Manufacturer" "Murata" (at 96.52 74.93 0)
+    (property "Part Number" "CL21A106KAYNNNE" (at 96.52 74.93 0)
+      (effects (font (size 1.27 1.27)) hide)
+    )
+    (property "Manufacturer" "Samsung Electro-Mechanics" (at 96.52 74.93 0)
       (effects (font (size 1.27 1.27)) hide)
     )
@@
       (effects (font (size 1.27 1.27)) hide)
     )
+    (property "LCSC Part" "C15850" (at 96.52 74.93 0)
+      (effects (font (size 1.27 1.27)) hide)
+    )
     (pin "1")
     (pin "2")
@@
       (effects (font (size 1.27 1.27)) (justify left))
     )
-    (property "Value" "1u/10V" (at 124.46 130.81 0)
+    (property "Value" "1u" (at 124.46 130.81 0)
       (effects (font (size 1.27 1.27)) (justify left))
     )
@@
       (effects (font (size 1.27 1.27)) hide)
     )
-    (property "Part Number" "CL05A105KP5NNNC" (at 120.65 129.54 0)
+    (property "Part Number" "CL05A105KA5NQNC" (at 120.65 129.54 0)
       (effects (font (size 1.27 1.27)) hide)
     )
@@
       (effects (font (size 1.27 1.27)) hide)
     )
+    (property "LCSC Part" "C52923" (at 120.65 129.54 0)
+      (effects (font (size 1.27 1.27)) hide)
+    )
     (pin "1")
     (pin "2")
@@
       (effects (font (size 1.27 1.27)) hide)
     )
+    (property "LCSC Part" "C8678" (at 86.36 69.85 0)
+      (effects (font (size 1.27 1.27)) hide)
+    )
     (pin "2")
     (pin "1")
@@
       (effects (font (size 1.27 1.27)) hide)
     )
+    (property "LCSC Part" "C25117" (at 189.23 134.62 0)
+      (effects (font (size 1.27 1.27)) hide)
+    )
     (pin "1")
     (pin "2")
@@
       (effects (font (size 1.27 1.27)) hide)
     )
-    (property "Part Number" "CL21A226MPQNNNE" (at 198.12 74.93 0)
+    (property "Part Number" "CL21A226MAQNNNE" (at 198.12 74.93 0)
       (effects (font (size 1.27 1.27)) hide)
     )
@@
       (effects (font (size 1.27 1.27)) hide)
     )
+    (property "LCSC Part" "C45783" (at 198.12 74.93 0)
+      (effects (font (size 1.27 1.27)) hide)
+    )
     (pin "1")
     (pin "2")
@@
       (effects (font (size 1.27 1.27)) hide)
     )
+    (property "LCSC Part" "C25750" (at 173.99 73.66 0)
+      (effects (font (size 1.27 1.27)) hide)
+    )
     (pin "1")
     (pin "2")
@@
       (effects (font (size 1.27 1.27)) hide)
     )
+    (property "LCSC Part" "C25768" (at 173.99 81.28 0)
+      (effects (font (size 1.27 1.27)) hide)
+    )
     (pin "1")
     (pin "2")
@@
       (effects (font (size 1.27 1.27)) hide)
     )
-    (property "Part Number" "CL21A226MPQNNNE" (at 185.42 74.93 0)
+    (property "Part Number" "CL21A226MAQNNNE" (at 185.42 74.93 0)
       (effects (font (size 1.27 1.27)) hide)
     )
@@
     )
     (property "Desc" "CAP CER 22u 10V 0805 low-ESR" (at 185.42 74.93 0)
+      (effects (font (size 1.27 1.27)) hide)
+    )
+    (property "LCSC Part" "C45783" (at 185.42 74.93 0)
       (effects (font (size 1.27 1.27)) hide)
     )
@@
       (effects (font (size 1.27 1.27)) hide)
     )
+    (property "LCSC Part" "C2286" (at 189.23 125.73 0)
+      (effects (font (size 1.27 1.27)) hide)
+    )
     (pin "2")
     (pin "1")
@@
       (effects (font (size 1.27 1.27)) hide)
     )
+    (property "LCSC Part" "C1525" (at 149.86 72.39 0)
+      (effects (font (size 1.27 1.27)) hide)
+    )
     (pin "1")
     (pin "2")
@@
   (symbol (lib_id "Device:C") (at 162.56 73.66 0) (unit 1)
     (in_bom yes) (on_board yes) (dnp no) (fields_autoplaced)
-    (property "Reference" "C308" (at 166.37 72.39 0)
+    (property "Reference" "C307" (at 166.37 72.39 0)
       (effects (font (size 1.27 1.27)) (justify left))
     )
@@
       (effects (font (size 1.27 1.27)) hide)
     )
-    (pin "2")
-    (pin "1")
-    (instances
-      (project "WG-Segment"
-        (path "/9a5339e6-f970-4986-a2cb-f70ab323b7e1/59659887-599e-4b15-819a-7d99a27b9ab4"
-          (reference "C308") (unit 1)
+    (property "LCSC Part" "C1546" (at 162.56 73.66 0)
+      (effects (font (size 1.27 1.27)) hide)
+    )
+    (pin "2")
+    (pin "1")
+    (instances
+      (project "WG-Segment"
+        (path "/9a5339e6-f970-4986-a2cb-f70ab323b7e1/59659887-599e-4b15-819a-7d99a27b9ab4"
+          (reference "C307") (unit 1)
         )
       )
@@
       (effects (font (size 1.27 1.27)) hide)
     )
+    (property "LCSC Part" "C2071868" (at 133.35 72.39 0)
+      (effects (font (size 1.27 1.27)) hide)
+    )
